File: thunderbolt-pcie-adapter.kicad_pcb (KiCad board)
At the start: 6 copper layers, 70 x 50 mm, 277 parts, among them J1 USB-C_JAE_DX07S024JJ2, J2 PCIe_x4_Conn_EdgeMount_Open, J3 Molex_Nano-Fit_1x2_1053131102, Q1 BC817-25W, Q2 BC817-25W, Q3 DZDH0401DW, Q4 DZDH0401DW, Q5 SI7613DN-T1-GE3, Q6 SI7613DN-T1-GE3, U1 LT8350RV, U2 MP2386GG, U3 TPS65983BAZBHR, U4 JHL6340SLLSQ, U5 MX25L8006EM1I-12G, U6 SI52112-B6-GT, Y1 Resonator_25MHz_ABM8G, Y2 Resonator_25MHz_ABM8G

Commit message: Measurement PCB: Add Kapton tape mask pieces for orientation on BGA footprint
These are the two main Kapton tape mask pieces used for soldering 0402 terminating resistors on PCIe_RX3 DPs.
I put them to make it easier to find the right pad on the footprint, among 300+ other ones.
Other:
- board text added: "Kapton Tape Mask"
Changed lines of the file:
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@@
 		(layer "F.SilkS")
+	)
+	(gr_poly
+		(pts
+			(xy 135.56 82.38) (xy 135.33 86.46) (xy 135.03 93.31) (xy 130.19 93.12) (xy 130.92 72.85) (xy 134.86 73.36)
+		)
+		(stroke
+			(width 0.15)
+			(type solid)
+		)
+		(fill none)
+		(layer "Dwgs.User")
+	)
+	(gr_poly
+		(pts
+			(xy 137.06 93.17) (xy 141.22 93.36) (xy 147.89 90.97) (xy 141.21 72.08) (xy 134.86 73.36) (xy 137.54 86.53)
+			(xy 137.45 89.4) (xy 137.44 89.39) (xy 137.06 93.18)
+		)
+		(stroke
+			(width 0.2)
+			(type solid)
+		)
+		(fill none)
+		(layer "Dwgs.User")
 	)
 	(gr_line
@@
 			)
 		)
+	)
+	(gr_text "Kapton\nTape\nMask"
+		(at 142.84 85.88 0)
+		(layer "Dwgs.User")
+		(effects
+			(font
+				(size 1.5 1)
+				(thickness 0.2)
+			)
+		)
+	)
+	(gr_text "Kapton\nTape\nMask"
+		(at 132.4 85.08 0)
+		(layer "Dwgs.User")
+		(effects
+			(font
+				(size 1.5 1)
+				(thickness 0.2)
+			)
+		)
