File: power.kicad_sch (KiCad schematic)
At the start: 128 parts, among them Q2 BC817-25W, Q3 DZDH0401DW, Q4 DZDH0401DW, Q5 SI7613DN-T1-GE3, Q6 SI7613DN-T1-GE3, U1 LT8350RV, U2 MP2386GG, U3 TPS65983BAZBHR

Commit message: SCH: Fix typo in Title Block, clarify authorship
Other:
- title: Thunderbolt PCIe Adaper -> Thunderbolt PCIe Adapter
Changed lines of the file:
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@@
 	(paper "A3")
 	(title_block
-		(title "Thunderbolt PCIe Adaper")
-		(date "2023-08-09")
+		(title "Thunderbolt PCIe Adapter")
+		(date "2025-07-04")
 		(rev "1.0.2")
-		(comment 1 "www.antmicro.com")
-		(comment 2 "Antmicro Ltd.")
+		(comment 1 "https://github.com/KataFF/tbt-pcie-adapter")
+		(comment 2 "Further modifications by Kajetan Wierszelis")
+		(comment 3 "www.antmicro.com")
+		(comment 4 "Original design (up to rev 1.0.2) by Antmicro Ltd.")
 	)
 	(junction
