File: tb.kicad_sch (KiCad schematic)
At the start: 67 parts, among them U4 JHL6340SLLSQ, U5 MX25L8006EM1I-12G, U6 SI52112-B6-GT, U7 MX25L8006EM2I-12G, Y1 Resonator_25MHz_ABM8G, Y2 Resonator_25MHz_ABM8G

Commit message: SCH: Fix typo in Title Block, clarify authorship
Other:
- title: Thunderbolt PCIe Adaper -> Thunderbolt PCIe Adapter
Changed lines of the file:
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@@
 	(paper "A3")
 	(title_block
-		(title "Thunderbolt PCIe Adaper")
-		(date "2023-08-09")
+		(title "Thunderbolt PCIe Adapter")
+		(date "2025-07-04")
 		(rev "1.0.2")
-		(comment 1 "www.antmicro.com")
-		(comment 2 "Antmicro Ltd.")
+		(comment 1 "https://github.com/KataFF/tbt-pcie-adapter")
+		(comment 2 "Further modifications by Kajetan Wierszelis")
+		(comment 3 "www.antmicro.com")
+		(comment 4 "Original design (up to rev 1.0.2) by Antmicro Ltd.")
 	)
 	(junction
