File: thunderbolt-pcie-adapter.kicad_sch (KiCad schematic)
At the start: 9 parts

Commit message: SCH: Fix typo in Title Block, clarify authorship
Other:
- title: Thunderbolt PCIe Adaper -> Thunderbolt PCIe Adapter
Changed lines of the file:
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@@
 	(paper "A3")
 	(title_block
-		(title "Thunderbolt PCIe Adaper")
-		(date "2025-05-09")
+		(title "Thunderbolt PCIe Adapter")
+		(date "2025-07-04")
 		(rev "1.0.3")
-		(comment 1 "www.antmicro.com")
-		(comment 2 "Original design (up to rev 1.0.2) by Antmicro, further modifications by Kajetan Wierszelis")
+		(comment 1 "https://github.com/KataFF/tbt-pcie-adapter")
+		(comment 2 "Further modifications by Kajetan Wierszelis")
+		(comment 3 "www.antmicro.com")
+		(comment 4 "Original design (up to rev 1.0.2) by Antmicro Ltd.")
 	)
 	(text "Thunderbolt - PCIe Adapter"
